Commit message: lab4 gazebo y ros2control agregado

File: lab3_urdf_rviz_gazebo/lab3_urdf_rviz_gazebo/urdf/1DOF-robot.urdf (robot description, URDF)
Before this commit: robot robot_name, 2 links, 1 joints
Joints:
- joint base_brazo_joint: limit lower=${-pi/2} upper=${pi/2} effort=100 velocity=100 -> lower=-1.5 upper=1.5 effort=100 velocity=100

File: lab4_gazebo/install/lab4_gazebo/share/lab4_gazebo/models/differential-robot.xacro (robot description, xacro)
@@ -1 +1,112 @@
-/home/sguajardo/UBB-ROS-2025/lab4_gazebo/build/lab4_gazebo/models/differential-robot.xacro
+<?xml version="1.0"?>
+<robot name="my_first_robot" xmlns:xacro="http://ros.org/wiki/xacro">
+  <xacro:property name="base_width" value = "0.31"/>
+  <xacro:property name="base_length" value = "0.42"/>
+  <xacro:property name="base_height" value = "0.18"/>
+  <xacro:property name="wheel_radius" value="0.10"/>
+  <xacro:property name="wheel_width" value="0.04"/>
+  <xacro:property name="wheel_ygap" value="0.025"/>
+  <xacro:property name="wheel_zoff" value="0.01"/>
+  <xacro:property name="wheel_xoff" value="0.05"/>
+  <xacro:property name="caster_xoff" value="0.1"/>
+  <!-- Macros de inercia -->
+  <xacro:macro name="box_inertia" params="m w h d">
+    <inertial>
+      <origin xyz="0 0 0" rpy="${pi/2} 0 ${pi/2}"/>
+      <mass value="${m}"/>
+      <inertia ixx="${(m/12) * (h*h + d*d)}" ixy="0.0" ixz="0.0" iyy="${(m/12) * (w*w + d*d)}" iyz="0.0" izz="${(m/12) * (w*w + h*h)}"/>
+    </inertial>
+  </xacro:macro>
+  <xacro:macro name="cylinder_inertia" params="m r h">
+    <inertial>
+      <origin xyz="0 0 0" rpy="${pi/2} 0 0" />
+      <mass value="${m}"/>
+      <inertia ixx="${(m/12) * (3*r*r + h*h)}" ixy = "0" ixz = "0" iyy="${(m/12) * (3*r*r + h*h)}" iyz = "0" izz="${(m/2) * (r*r)}"/>
+    </inertial>
+  </xacro:macro>
+  <xacro:macro name="sphere_inertia" params="m r">
+    <inertial>
+      <mass value="${m}"/>
+      <inertia ixx="${(2/5) * m * (r*r)}" ixy="0.0" ixz="0.0" iyy="${(2/5) * m * (r*r)}" iyz="0.0" izz="${(2/5) * m * (r*r)}"/>
+    </inertial>
+  </xacro:macro>
+  <!-- Eslabón Ficticio para referencia de Gazebo -->
+  <link name="base_footprint">
+  </link>
+  <!-- Robot Base -->
+  <link name="base_link">
+    <visual>
+    <origin xyz="0 0 ${base_height/2}" rpy="0 0 0"/>
+      <geometry>
+        <box size="${base_length} ${base_width} ${base_height}"/>
+      </geometry>
+      <material name="Cyan">
+        <color rgba="0 1.0 1.0 1.0"/>
+      </material>
+    </visual>
+    <collision>
+    <origin xyz="0 0 ${base_height/2}" rpy="0 0 0"/>
+      <geometry>
+        <box size="${base_length} ${base_width} ${base_height}"/>
+      </geometry>
+    </collision>
+    <xacro:box_inertia m="5" w="${base_width}" d="${base_length}" h="${base_height}"/>
+  </link>
+  <joint name="base_link_joint" type="fixed">
+    <parent link="base_footprint"/>
+    <child link="base_link"/>
+  </joint>
+  <!-- Caster Wheel -->
+  <link name="caster">
+    <visual>
+      <geometry>
+        <sphere radius="${wheel_zoff}"/>
+      </geometry>
+      <material name="white">
+        <color rgba="1 1.0 1.0 1.0"/>
+      </material>
+    </visual>
+    <collision>
+      <origin xyz="0 0 0" rpy="0 0 0"/>
+      <geometry>
+        <sphere radius="${wheel_zoff}"/>
+      </geometry>
+    </collision>
+    <xacro:sphere_inertia m="0.5" r="${(wheel_radius+wheel_zoff-(base_height/2))}"/>
+  </link>
+  <joint name="caster_joint" type="fixed">
+    <parent link="base_link"/>
+    <child link="caster"/>
+    <origin xyz="${-caster_xoff} 0.0 0" rpy="0 0 0"/>
+  </joint>
+  <!-- Wheels -->
+  <xacro:macro name="wheel" params="prefix x_reflect y_reflect">
+    <link name="${prefix}_link">
+      <visual>
+        <origin xyz="0 0 0" rpy="${pi/2} 0 0"/>
+        <geometry>
+            <cylinder radius="${wheel_radius}" length="${wheel_width}"/>
+        </geometry>
+        <material name="Gray">
+          <color rgba="0.5 0.5 0.5 1.0"/>
+        </material>
+      </visual>
+      <collision>
+        <origin xyz="0 0 0" rpy="${pi/2} 0 0"/>
+        <geometry>
+          <cylinder radius="${wheel_radius}" length="${wheel_width}"/>
+        </geometry>
+      </collision>
+      <xacro:cylinder_inertia m="0.5" r="${wheel_radius}" h="${wheel_width}"/>
+    </link>
+    <joint name="${prefix}_joint" type="continuous">
+      <parent link="base_link"/>
+      <child link="${prefix}_link"/>
+      <origin xyz="${-x_reflect*wheel_xoff} ${y_reflect*(base_width/2+wheel_ygap)} ${wheel_radius-wheel_zoff}" rpy="0 0 0"/>
+      <axis xyz="0 1 0"/>
+    </joint>
+  </xacro:macro>
+  <xacro:wheel prefix="drivewhl_l" x_reflect="-1" y_reflect="1" />
+  <xacro:wheel prefix="drivewhl_r" x_reflect="-1" y_reflect="-1" />
+  <xacro:include filename="differential-robot.gazebo.urdf"/>
+</robot>
